File: pcb/pcb.kicad_sch (KiCad schematic)
At the start: 20 parts

Commit message: Rework GDT_AC as SMT using back sire WIRE_B only
Parts:
- GDT_AC: value B5G470L -> SMD5050-470NA; footprint DogFence:B5G470L_P15.24mm_NS_Overpass -> DogFence:SMD5050-470NA; LCSC C5337217 -> C39692533; MPN B5G470L -> SMD5050-470NA; Manufacturer Bencent -> Ruilon
Other:
- note added: "(6.00mm B.Cu rail below)"
- note added: "SMT GDT_AC: A to C"
- note removed: "(>=2.0mm air gap standoff)"
- note removed: "Axial GDT_AC bridges Wire B"
Changed lines of the file:
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@@
 		)
 	)
-	(text "Axial GDT_AC bridges Wire B"
+	(text "SMT GDT_AC: A to C"
 		(exclude_from_sim no)
 		(at 91.44 97.65 0)
@@
 		)
 	)
-	(text "(>=2.0mm air gap standoff)"
+	(text "(6.00mm B.Cu rail below)"
 		(exclude_from_sim no)
 		(at 91.44 100.65 0)
@@
 		(dnp no)
 		(property "Reference" "GDT_AC"
-			(at 118.8 76.2 90)
+			(at 111 76.2 90)
 			(effects
 				(font
@@
 					(bold yes)
 				)
-				(justify left)
-			)
-		)
-		(property "Value" "B5G470L"
-			(at 118.8 78.74 90)
+				(justify right)
+			)
+		)
+		(property "Value" "SMD5050-470NA"
+			(at 111 78.74 90)
 			(effects
 				(font
 					(size 1.016 1.016)
 				)
-				(justify left)
+				(justify right)
 			)
 		)
@@
 			)
 		)
-		(property "Manufacturer" "Bencent"
+		(property "Manufacturer" "Ruilon"
 			(at 114.3 77.47 0)
 			(effects
@@
 			)
 		)
-		(property "Footprint" "DogFence:B5G470L_P15.24mm_NS_Overpass"
+		(property "Footprint" "DogFence:SMD5050-470NA"
 			(at 114.3 77.47 90)
 			(effects
@@
 			)
 		)
-		(property "Datasheet" "https://www.lcsc.com/datasheet/C5337217.pdf"
+		(property "Datasheet" "https://www.lcsc.com/datasheet/C39692533.pdf"
 			(at 114.3 77.47 0)
 			(effects
@@
 			)
 		)
-		(property "MPN" "B5G470L"
+		(property "MPN" "SMD5050-470NA"
 			(at 114.3 77.47 0)
 			(effects
@@
 			)
 		)
-		(property "LCSC" "C5337217"
+		(property "LCSC" "C39692533"
 			(at 114.3 77.47 0)
 			(effects
